Commit message: Added basic differential drive controller for wheels (temporary solution)

File: catkin_ws/src/bricklayer_gazebo/models/youbot/model.urdf (robot description, URDF)
Before this commit: robot youbot, 21 links, 20 joints
Joints:
- joint caster_joint_bl: type continuous -> fixed
- joint caster_joint_br: type continuous -> fixed
- joint caster_joint_fl: type continuous -> fixed
- joint caster_joint_fr: type continuous -> fixed
- joint wheel_joint_bl: limit lower=0.0 upper=0.0 effort=1.0 velocity=0.0 -> (none)
- joint wheel_joint_br: limit lower=0.0 upper=0.0 effort=1.0 velocity=0.0 -> (none)
- joint wheel_joint_fl: limit lower=0.0 upper=0.0 effort=1.0 velocity=0.0 -> (none)
- joint wheel_joint_fr: limit lower=0.0 upper=0.0 effort=1.0 velocity=0.0 -> (none)
