Commit message: Renamed bricklayer to paintbot

File: catkin_ws/src/paintbot_gazebo/models/paintbot/paintbot.urdf (robot description, URDF)
Before this commit: robot youbot, 21 links, 20 joints
Links:
- link arm_link_0: geometry collision mesh filename=package://paintbot_gazebo/models/paintbot/meshes/arm/arm0_c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 scale=1.0 1.0 1.0; visual mesh filename=package://paintbot_gazebo/models/paintbot/meshes/arm/arm0.d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 scale=1.0 1.0 1.0
- link arm_link_1: geometry collision mesh filename=package://paintbot_gazebo/models/paintbot/meshes/arm/arm1_c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 scale=1.0 1.0 1.0; visual mesh filename=package://paintbot_gazebo/models/paintbot/meshes/arm/arm1.d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 scale=1.0 1.0 1.0
- link arm_link_2: geometry collision mesh filename=package://paintbot_gazebo/models/paintbot/meshes/arm/arm2_c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 scale=1.0 1.0 1.0; visual mesh filename=package://paintbot_gazebo/models/paintbot/meshes/arm/arm2.d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 scale=1.0 1.0 1.0
- link arm_link_3: geometry collision mesh filename=package://paintbot_gazebo/models/paintbot/meshes/arm/arm3_c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 scale=1.0 1.0 1.0; visual mesh filename=package://paintbot_gazebo/models/paintbot/meshes/arm/arm3.d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 scale=1.0 1.0 1.0
- link arm_link_4: geometry collision mesh filename=package://paintbot_gazebo/models/paintbot/meshes/arm/arm4_c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 scale=1.0 1.0 1.0; visual mesh filename=package://paintbot_gazebo/models/paintbot/meshes/arm/arm4.d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 scale=1.0 1.0 1.0
- link arm_link_5: geometry collision mesh filename=package://paintbot_gazebo/models/paintbot/meshes/arm/arm5_c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 scale=1.0 1.0 1.0; visual mesh filename=package://paintbot_gazebo/models/paintbot/meshes/arm/arm5.d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 scale=1.0 1.0 1.0
- link base_laser_front_link: geometry collision mesh filename=package://paintbot_gazebo/models/paintbot/meshes/laser/hoku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 scale=1.0 1.0 1.0; visual mesh filename=package://paintbot_gazebo/models/paintbot/meshes/laser/hoku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 scale=1.0 1.0 1.0
- link base_link: geometry collision mesh filename=package://paintbot_gazebo/models/paintbot/meshes/base/base_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 scale=1.0 1.0 1.0; visual mesh filename=package://paintbot_gazebo/models/paintbot/meshes/base/base.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 scale=1.0 1.0 1.0
- link gripper_finger_link_l: geometry collision mesh filename=package://paintbot_gazebo/models/paintbot/meshes/gripper/fi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 scale=1.0 1.0 1.0; visual mesh filename=package://paintbot_gazebo/models/paintbot/meshes/gripper/fi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 scale=1.0 1.0 1.0
- link gripper_finger_link_r: geometry collision mesh filename=package://paintbot_gazebo/models/paintbot/meshes/gripper/fi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 scale=1.0 1.0 1.0; visual mesh filename=package://paintbot_gazebo/models/paintbot/meshes/gripper/fi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 scale=1.0 1.0 1.0
- link gripper_palm_link: geometry collision mesh filename=package://paintbot_gazebo/models/paintbot/meshes/gripper/pa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 scale=1.0 1.0 1.0; visual mesh filename=package://paintbot_gazebo/models/paintbot/meshes/gripper/pa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 scale=1.0 1.0 1.0
- link plate_link: geometry collision mesh filename=package://paintbot_gazebo/models/paintbot/meshes/plate/plat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 scale=1.0 1.0 1.0; visual mesh filename=package://paintbot_gazebo/models/paintbot/meshes/plate/plat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 scale=1.0 1.0 1.0
- link wheel_link_bl: geometry collision cylinder length=0.005000 radius=0.050000; visual mesh filename=package://paintbot_gazebo/models/paintbot/meshes/base/back-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 scale=1.0 1.0 1.0
- link wheel_link_br: geometry collision cylinder length=0.005000 radius=0.050000; visual mesh filename=package://paintbot_gazebo/models/paintbot/meshes/base/back-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 scale=1.0 1.0 1.0
- link wheel_link_fl: geometry collision cylinder length=0.005000 radius=0.050000; visual mesh filename=package://paintbot_gazebo/models/paintbot/meshes/base/front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 scale=1.0 1.0 1.0
- link wheel_link_fr: geometry collision cylinder length=0.005000 radius=0.050000; visual mesh filename=package://paintbot_gazebo/models/paintbot/meshes/base/front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 scale=1.0 1.0 1.0
