Commit message: Initial integration of MoveIt with main nodes

File: catkin_ws/src/paintbot_description/urdf/paintbot_mi.urdf (robot description, URDF)
Before this commit: robot paintbot, 22 links, 21 joints
Joints:
- removed joint virtual_joint
- added joint virtual_base_joint: type fixed, parent virtual_base, child base_footprint
