Commit message: Moved paintbot description to paintbot_description package

File: catkin_ws/src/paintbot_description/urdf/paintbot.urdf (robot description, URDF)
Before this commit: robot paintbot, 21 links, 20 joints
Links:
- link arm_link_0: geometry collision mesh filename=package://paintbot_description/meshes/arm/arm0_convex.stl scale=1.0 1.0 1.0; visual mesh filename=package://paintbot_description/meshes/arm/arm0.dae scale=1.0 1.0 1.0
- link arm_link_1: geometry collision mesh filename=package://paintbot_description/meshes/arm/arm1_convex.stl scale=1.0 1.0 1.0; visual mesh filename=package://paintbot_description/meshes/arm/arm1.dae scale=1.0 1.0 1.0
- link arm_link_2: geometry collision mesh filename=package://paintbot_description/meshes/arm/arm2_convex.stl scale=1.0 1.0 1.0; visual mesh filename=package://paintbot_description/meshes/arm/arm2.dae scale=1.0 1.0 1.0
- link arm_link_3: geometry collision mesh filename=package://paintbot_description/meshes/arm/arm3_convex.stl scale=1.0 1.0 1.0; visual mesh filename=package://paintbot_description/meshes/arm/arm3.dae scale=1.0 1.0 1.0
- link arm_link_4: geometry collision mesh filename=package://paintbot_description/meshes/arm/arm4_convex.stl scale=1.0 1.0 1.0; visual mesh filename=package://paintbot_description/meshes/arm/arm4.dae scale=1.0 1.0 1.0
- link arm_link_5: geometry collision mesh filename=package://paintbot_description/meshes/arm/arm5_convex.stl scale=1.0 1.0 1.0; visual mesh filename=package://paintbot_description/meshes/arm/arm5.dae scale=1.0 1.0 1.0
- link base_laser_front_link: geometry collision mesh filename=package://paintbot_description/meshes/laser/hokuyo_convex.s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 scale=1.0 1.0 1.0; visual mesh filename=package://paintbot_description/meshes/laser/hokuyo.dae scale=1.0 1.0 1.0
- link base_link: geometry collision mesh filename=package://paintbot_description/meshes/base/base_convex.stl scale=1.0 1.0 1.0; visual mesh filename=package://paintbot_description/meshes/base/base.dae scale=1.0 1.0 1.0
- link gripper_finger_link_l: geometry collision mesh filename=package://paintbot_description/meshes/gripper/finger_convex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 scale=1.0 1.0 1.0; visual mesh filename=package://paintbot_description/meshes/gripper/finger.stl scale=1.0 1.0 1.0
- link gripper_finger_link_r: geometry collision mesh filename=package://paintbot_description/meshes/gripper/finger_convex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 scale=1.0 1.0 1.0; visual mesh filename=package://paintbot_description/meshes/gripper/finger.stl scale=1.0 1.0 1.0
- link gripper_palm_link: geometry collision mesh filename=package://paintbot_description/meshes/gripper/palm_convex.s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 scale=1.0 1.0 1.0; visual mesh filename=package://paintbot_description/meshes/gripper/palm.stl scale=1.0 1.0 1.0
- link plate_link: geometry collision mesh filename=package://paintbot_description/meshes/plate/plate_convex.stl scale=1.0 1.0 1.0; visual mesh filename=package://paintbot_description/meshes/plate/plate.dae scale=1.0 1.0 1.0
- link wheel_link_bl: geometry collision cylinder length=0.005000 radius=0.050000; visual mesh filename=package://paintbot_description/meshes/base/back-left_wheel.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 scale=1.0 1.0 1.0
- link wheel_link_br: geometry collision cylinder length=0.005000 radius=0.050000; visual mesh filename=package://paintbot_description/meshes/base/back-right_wheel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 scale=1.0 1.0 1.0
- link wheel_link_fl: geometry collision cylinder length=0.005000 radius=0.050000; visual mesh filename=package://paintbot_description/meshes/base/front-left_wheel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 scale=1.0 1.0 1.0
- link wheel_link_fr: geometry collision cylinder length=0.005000 radius=0.050000; visual mesh filename=package://paintbot_description/meshes/base/front-right_whee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 scale=1.0 1.0 1.0

Commit message: Temporary work around for wheel values

File: catkin_ws/src/paintbot_description/urdf/paintbot.urdf (robot description, URDF)
Before this commit: robot paintbot, 21 links, 20 joints
Links:
- link wheel_link_bl: mass 0.400000 -> 1.000000; geometry collision cylinder length=0.100000 radius=0.075000; visual mesh filename=package://paintbot_description/meshes/base/back-left_wheel.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 scale=1.0 1.0 1.0
- link wheel_link_br: mass 0.400000 -> 1.000000; geometry collision cylinder length=0.100000 radius=0.075000; visual mesh filename=package://paintbot_description/meshes/base/back-right_wheel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 scale=1.0 1.0 1.0
- link wheel_link_fl: mass 0.400000 -> 1.000000; geometry collision cylinder length=0.100000 radius=0.075000; visual mesh filename=package://paintbot_description/meshes/base/front-left_wheel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 scale=1.0 1.0 1.0
- link wheel_link_fr: mass 0.400000 -> 1.000000; geometry collision cylinder length=0.100000 radius=0.075000; visual mesh filename=package://paintbot_description/meshes/base/front-right_whee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 scale=1.0 1.0 1.0

Commit message: MoveIt Poc

File: catkin_ws/src/paintbot_description/urdf/paintbot.urdf (robot description, URDF)
Before this commit: robot paintbot, 21 links, 20 joints
Links:
- added link virtual_base
Joints:
- added joint virtual_joint: type fixed, parent virtual_base, child base_footprint

Commit message: Modified logging output; Moved paintbot_description/meshes into paintbot_description/urdf; Removed paintbot_description/materials

File: catkin_ws/src/paintbot_description/urdf/paintbot.urdf (robot description, URDF)
Before this commit: robot paintbot, 22 links, 21 joints
Links:
- link arm_link_0: geometry collision mesh filename=package://paintbot_description/urdf/meshes/arm/arm0_convex.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 scale=1.0 1.0 1.0; visual mesh filename=package://paintbot_description/urdf/meshes/arm/arm0.dae scale=1.0 1.0 1.0
- link arm_link_1: geometry collision mesh filename=package://paintbot_description/urdf/meshes/arm/arm1_convex.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 scale=1.0 1.0 1.0; visual mesh filename=package://paintbot_description/urdf/meshes/arm/arm1.dae scale=1.0 1.0 1.0
- link arm_link_2: geometry collision mesh filename=package://paintbot_description/urdf/meshes/arm/arm2_convex.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 scale=1.0 1.0 1.0; visual mesh filename=package://paintbot_description/urdf/meshes/arm/arm2.dae scale=1.0 1.0 1.0
- link arm_link_3: geometry collision mesh filename=package://paintbot_description/urdf/meshes/arm/arm3_convex.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 scale=1.0 1.0 1.0; visual mesh filename=package://paintbot_description/urdf/meshes/arm/arm3.dae scale=1.0 1.0 1.0
- link arm_link_4: geometry collision mesh filename=package://paintbot_description/urdf/meshes/arm/arm4_convex.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 scale=1.0 1.0 1.0; visual mesh filename=package://paintbot_description/urdf/meshes/arm/arm4.dae scale=1.0 1.0 1.0
- link arm_link_5: geometry collision mesh filename=package://paintbot_description/urdf/meshes/arm/arm5_convex.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 scale=1.0 1.0 1.0; visual mesh filename=package://paintbot_description/urdf/meshes/arm/arm5.dae scale=1.0 1.0 1.0
- link base_laser_front_link: geometry collision mesh filename=package://paintbot_description/urdf/meshes/laser/hokuyo_con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 scale=1.0 1.0 1.0; visual mesh filename=package://paintbot_description/urdf/meshes/laser/hokuyo.dae scale=1.0 1.0 1.0
- link base_link: geometry collision mesh filename=package://paintbot_description/urdf/meshes/base/base_convex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 scale=1.0 1.0 1.0; visual mesh filename=package://paintbot_description/urdf/meshes/base/base.dae scale=1.0 1.0 1.0
- link gripper_finger_link_l: geometry collision mesh filename=package://paintbot_description/urdf/meshes/gripper/finger_c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 scale=1.0 1.0 1.0; visual mesh filename=package://paintbot_description/urdf/meshes/gripper/finger.s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 scale=1.0 1.0 1.0
- link gripper_finger_link_r: geometry collision mesh filename=package://paintbot_description/urdf/meshes/gripper/finger_c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 scale=1.0 1.0 1.0; visual mesh filename=package://paintbot_description/urdf/meshes/gripper/finger.s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 scale=1.0 1.0 1.0
- link gripper_palm_link: geometry collision mesh filename=package://paintbot_description/urdf/meshes/gripper/palm_con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 scale=1.0 1.0 1.0; visual mesh filename=package://paintbot_description/urdf/meshes/gripper/palm.stl scale=1.0 1.0 1.0
- link plate_link: geometry collision mesh filename=package://paintbot_description/urdf/meshes/plate/plate_conv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 scale=1.0 1.0 1.0; visual mesh filename=package://paintbot_description/urdf/meshes/plate/plate.dae scale=1.0 1.0 1.0
- link wheel_link_bl: geometry collision cylinder length=0.100000 radius=0.075000; visual mesh filename=package://paintbot_description/urdf/meshes/base/back-left_w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 scale=1.0 1.0 1.0
- link wheel_link_br: geometry collision cylinder length=0.100000 radius=0.075000; visual mesh filename=package://paintbot_description/urdf/meshes/base/back-right_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 scale=1.0 1.0 1.0
- link wheel_link_fl: geometry collision cylinder length=0.100000 radius=0.075000; visual mesh filename=package://paintbot_description/urdf/meshes/base/front-left_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 scale=1.0 1.0 1.0
- link wheel_link_fr: geometry collision cylinder length=0.100000 radius=0.075000; visual mesh filename=package://paintbot_description/urdf/meshes/base/front-right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 scale=1.0 1.0 1.0

File: catkin_ws/src/paintbot_description/urdf/paintbot_mi.urdf (robot description, URDF)
Before this commit: robot paintbot, 22 links, 21 joints
Links:
- link arm_link_0: geometry collision mesh filename=package://paintbot_description/urdf/meshes/arm/arm0_convex.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 scale=1.0 1.0 1.0; visual mesh filename=package://paintbot_description/urdf/meshes/arm/arm0.dae scale=1.0 1.0 1.0
- link arm_link_1: geometry collision mesh filename=package://paintbot_description/urdf/meshes/arm/arm1_convex.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 scale=1.0 1.0 1.0; visual mesh filename=package://paintbot_description/urdf/meshes/arm/arm1.dae scale=1.0 1.0 1.0
- link arm_link_2: geometry collision mesh filename=package://paintbot_description/urdf/meshes/arm/arm2_convex.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 scale=1.0 1.0 1.0; visual mesh filename=package://paintbot_description/urdf/meshes/arm/arm2.dae scale=1.0 1.0 1.0
- link arm_link_3: geometry collision mesh filename=package://paintbot_description/urdf/meshes/arm/arm3_convex.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 scale=1.0 1.0 1.0; visual mesh filename=package://paintbot_description/urdf/meshes/arm/arm3.dae scale=1.0 1.0 1.0
- link arm_link_4: geometry collision mesh filename=package://paintbot_description/urdf/meshes/arm/arm4_convex.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 scale=1.0 1.0 1.0; visual mesh filename=package://paintbot_description/urdf/meshes/arm/arm4.dae scale=1.0 1.0 1.0
- link arm_link_5: geometry collision mesh filename=package://paintbot_description/urdf/meshes/arm/arm5_convex.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 scale=1.0 1.0 1.0; visual mesh filename=package://paintbot_description/urdf/meshes/arm/arm5.dae scale=1.0 1.0 1.0
- link base_laser_front_link: geometry collision mesh filename=package://paintbot_description/urdf/meshes/laser/hokuyo_con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 scale=1.0 1.0 1.0; visual mesh filename=package://paintbot_description/urdf/meshes/laser/hokuyo.dae scale=1.0 1.0 1.0
- link base_link: geometry collision mesh filename=package://paintbot_description/urdf/meshes/base/base_convex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 scale=1.0 1.0 1.0; visual mesh filename=package://paintbot_description/urdf/meshes/base/base.dae scale=1.0 1.0 1.0
- link gripper_finger_link_l: geometry collision mesh filename=package://paintbot_description/urdf/meshes/gripper/finger_c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 scale=1.0 1.0 1.0; visual mesh filename=package://paintbot_description/urdf/meshes/gripper/finger.s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 scale=1.0 1.0 1.0
- link gripper_finger_link_r: geometry collision mesh filename=package://paintbot_description/urdf/meshes/gripper/finger_c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 scale=1.0 1.0 1.0; visual mesh filename=package://paintbot_description/urdf/meshes/gripper/finger.s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 scale=1.0 1.0 1.0
- link gripper_palm_link: geometry collision mesh filename=package://paintbot_description/urdf/meshes/gripper/palm_con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 scale=1.0 1.0 1.0; visual mesh filename=package://paintbot_description/urdf/meshes/gripper/palm.stl scale=1.0 1.0 1.0
- link plate_link: geometry collision mesh filename=package://paintbot_description/urdf/meshes/plate/plate_conv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 scale=1.0 1.0 1.0; visual mesh filename=package://paintbot_description/meshes/plate/plate.dae scale=1.0 1.0 1.0
- link wheel_link_bl: geometry collision cylinder length=0.100000 radius=0.075000; visual mesh filename=package://paintbot_description/urdf/meshes/base/back-left_w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 scale=1.0 1.0 1.0
- link wheel_link_br: geometry collision cylinder length=0.100000 radius=0.075000; visual mesh filename=package://paintbot_description/urdf/meshes/base/back-right_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 scale=1.0 1.0 1.0
- link wheel_link_fl: geometry collision cylinder length=0.100000 radius=0.075000; visual mesh filename=package://paintbot_description/urdf/meshes/base/front-left_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 scale=1.0 1.0 1.0
- link wheel_link_fr: geometry collision cylinder length=0.100000 radius=0.075000; visual mesh filename=package://paintbot_description/urdf/meshes/base/front-right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 scale=1.0 1.0 1.0

Commit message: Renamed paintbot_mi.urdf to paintbot.urdf; Removed mi_test.py and mi_test.launch

File: catkin_ws/src/paintbot_description/urdf/paintbot.urdf (robot description, URDF)
Before this commit: robot paintbot, 22 links, 21 joints
Links:
- link plate_link: geometry collision mesh filename=package://paintbot_description/urdf/meshes/plate/plate_conv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 scale=1.0 1.0 1.0; visual mesh filename=package://paintbot_description/meshes/plate/plate.dae scale=1.0 1.0 1.0
Joints:
- removed joint virtual_joint
- added joint virtual_base_joint: type fixed, parent virtual_base, child base_footprint

Commit message: Initial workin implementation of planar movement plugin

File: catkin_ws/src/paintbot_description/urdf/paintbot.urdf (robot description, URDF)
Before this commit: robot paintbot, 22 links, 21 joints
Links:
- removed link caster_link_bl
- removed link caster_link_br
- removed link caster_link_fl
- removed link caster_link_fr
Joints:
- removed joint caster_joint_bl
- removed joint caster_joint_br
- removed joint caster_joint_fl
- removed joint caster_joint_fr
- joint wheel_joint_bl: origin xyz=0  0  0 rpy=0  0  0 -> xyz=-0.228  0.158 -0.034 rpy=0  0  0; parent caster_link_bl -> base_link
- joint wheel_joint_br: origin xyz=0  0  0 rpy=0  0  0 -> xyz=-0.228 -0.158 -0.034 rpy=0  0  0; parent caster_link_br -> base_link
- joint wheel_joint_fl: origin xyz=0  0  0 rpy=0  0  0 -> xyz=0.228  0.158 -0.034 rpy=0  0  0; parent caster_link_fl -> base_link
- joint wheel_joint_fr: origin xyz=0  0  0 rpy=0  0  0 -> xyz=0.228 -0.158 -0.034 rpy=0  0  0; parent caster_link_fr -> base_link

Commit message: Navigation stack WIP

File: catkin_ws/src/paintbot_description/urdf/paintbot.urdf (robot description, URDF)
Before this commit: robot paintbot, 18 links, 17 joints
Joints:
- joint virtual_base_joint: origin (none) -> xyz=0 0 0 rpy=0 0 0

Commit message: Fixing two startup warnings

File: catkin_ws/src/paintbot_description/urdf/paintbot.urdf (robot description, URDF)
Before this commit: robot paintbot, 18 links, 17 joints
Links:
- link plate_link: geometry collision mesh filename=package://paintbot_description/urdf/meshes/plate/plate_conv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 scale=1.0 1.0 1.0; visual mesh filename=package://paintbot_description/urdf/meshes/plate/plate.dae scale=1.0 1.0 1.0

Commit message: Fixed paintbot wheel dimensions

File: catkin_ws/src/paintbot_description/urdf/paintbot.urdf (robot description, URDF)
Before this commit: robot paintbot, 18 links, 17 joints
Links:
- link wheel_link_bl: geometry collision cylinder length=0.072500 radius=0.050000; visual mesh filename=package://paintbot_description/urdf/meshes/base/back-left_w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 scale=1.0 1.0 1.0
- link wheel_link_br: geometry collision cylinder length=0.072500 radius=0.050000; visual mesh filename=package://paintbot_description/urdf/meshes/base/back-right_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 scale=1.0 1.0 1.0
- link wheel_link_fl: geometry collision cylinder length=0.072500 radius=0.050000; visual mesh filename=package://paintbot_description/urdf/meshes/base/front-left_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 scale=1.0 1.0 1.0
- link wheel_link_fr: geometry collision cylinder length=0.072500 radius=0.050000; visual mesh filename=package://paintbot_description/urdf/meshes/base/front-right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 scale=1.0 1.0 1.0
Joints:
- joint virtual_base_joint: origin xyz=0 0 0 rpy=0 0 0 -> (none)

Commit message: WIP: Adding roller to Paintbot model

File: catkin_ws/src/paintbot_description/urdf/paintbot.urdf (robot description, URDF)
Before this commit: robot paintbot, 18 links, 17 joints
Links:
- removed link gripper_finger_link_l
- removed link gripper_finger_link_r
- added link roller, mass 1; collision cylinder length=0.2286 radius=0.0254; visual cylinder length=0.2286 radius=0.0254
- added link roller_frame, mass 1; collision cylinder length=0.1524 radius=0.00635; visual cylinder length=0.1524 radius=0.00635
Joints:
- removed joint gripper_finger_joint_l
- removed joint gripper_finger_joint_r
- added joint roller_frame_joint: type fixed, parent gripper_palm_link, child roller_frame, origin xyz=0   0   0.09 rpy=0 0 0, axis 0 0 0, limit lower=0 upper=0 effort=0 velocity=0
- added joint roller_joint: type continuous, parent roller_frame, child roller, origin xyz=0  0  0.1 rpy=1.57079 0      0, axis 0  1  0

Commit message: Adjusted roller model; Load skill works with roller

File: catkin_ws/src/paintbot_description/urdf/paintbot.urdf (robot description, URDF)
Before this commit: robot paintbot, 18 links, 17 joints
Links:
- removed link roller_frame
Joints:
- removed joint roller_frame_joint
- joint roller_joint: axis 0  1  0 -> 0  0  0; limit (none) -> lower=0 upper=0 effort=0 velocity=0; origin xyz=0  0  0.1 rpy=1.57079 0      0 -> xyz=0  0  0.054 rpy=1.57079 0      0; parent roller_frame -> gripper_palm_link; type continuous -> fixed
